File: PGA-103+ LNA Mod2/PGA-103+ LNA Mod2.brd (EAGLE design)
At the start: 97.8 x 53 mm, 44 parts, among them IC1 7805DT, K1 G2RE, K2 G2RE, K3 G2RE, K4 G2RE, X1 SMA, X2 SMA

Commit message: Revalue the components
Parts:
- C1, C10: value 10n -> 10p
- C11, C15: value 1n -> 10n
- C13: value 10n -> 1n
- C16: value 1n -> 100n
- C3, C5, C7, C9: value 330p -> 22p
- C4: value 1n -> 10u
- C6: value 10n -> 3p3
- R1, R2: value 1u -> 90nH
- R3, R6: value 1u -> 1uH
Changed lines of the file:
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@@
 </autorouter>
 <elements>
-<element name="C1" library="rcl" package="C1206" value="10n" x="34.29" y="35.56" rot="R270"/>
-<element name="C10" library="rcl" package="C1206" value="10n" x="52.07" y="35.56" rot="R90"/>
-<element name="C11" library="rcl" package="C1206" value="1n" x="65.405" y="24.13"/>
+<element name="C1" library="rcl" package="C1206" value="10p" x="34.29" y="35.56" rot="R270"/>
+<element name="C10" library="rcl" package="C1206" value="10p" x="52.07" y="35.56" rot="R90"/>
+<element name="C11" library="rcl" package="C1206" value="10n" x="65.405" y="24.13"/>
 <element name="C12" library="rcl" package="C1206" value="330p" x="50.8" y="24.13"/>
-<element name="C13" library="rcl" package="C1206" value="10n" x="62.23" y="36.83"/>
+<element name="C13" library="rcl" package="C1206" value="1n" x="62.23" y="36.83"/>
 <element name="C14" library="rcl" package="C1206" value="1n" x="65.405" y="26.67" rot="R180"/>
 <element name="C2" library="rcl" package="C1206" value="1n" x="45.72" y="23.1775" rot="R90"/>
-<element name="C3" library="rcl" package="C1206" value="330p" x="34.29" y="30.48" rot="R90"/>
-<element name="C4" library="rcl" package="C1206" value="1n" x="43.18" y="23.1775" rot="R90"/>
-<element name="C5" library="rcl" package="C1206" value="330p" x="41.91" y="30.48" rot="R90"/>
-<element name="C6" library="rcl" package="C1206" value="10n" x="43.18" y="34.29"/>
-<element name="C7" library="rcl" package="C1206" value="330p" x="44.45" y="30.48" rot="R90"/>
+<element name="C3" library="rcl" package="C1206" value="22p" x="34.29" y="30.48" rot="R90"/>
+<element name="C4" library="rcl" package="C1206" value="10u" x="43.18" y="23.1775" rot="R90"/>
+<element name="C5" library="rcl" package="C1206" value="22p" x="41.91" y="30.48" rot="R90"/>
+<element name="C6" library="rcl" package="C1206" value="3p3" x="43.18" y="34.29"/>
+<element name="C7" library="rcl" package="C1206" value="22p" x="44.45" y="30.48" rot="R90"/>
 <element name="C8" library="rcl" package="B/3528-21R" value="10u" x="60.6425" y="13.335" rot="R270"/>
-<element name="C9" library="rcl" package="C1206" value="330p" x="52.07" y="30.48" rot="R90"/>
+<element name="C9" library="rcl" package="C1206" value="22p" x="52.07" y="30.48" rot="R90"/>
 <element name="D1" library="diode" package="DO35-7" value="1N4xxx" x="45.72" y="15.24" rot="R270"/>
 <element name="D2" library="diode" package="DO35-7" value="1N4xxx" x="31.75" y="15.24" rot="R270"/>
@@
 <attribute name="MPN" value="" x="83.82" y="46.99" size="1.778" layer="27" display="off"/>
 </element>
-<element name="R1" library="rcl" package="M1206" value="1u" x="38.1" y="34.29" rot="R180"/>
-<element name="R2" library="rcl" package="M1206" value="1u" x="48.26" y="34.29" rot="R180"/>
-<element name="R3" library="rcl" package="M1206" value="1u" x="55.245" y="30.48" rot="R90"/>
+<element name="R1" library="rcl" package="M1206" value="90nH" x="38.1" y="34.29" rot="R180"/>
+<element name="R2" library="rcl" package="M1206" value="90nH" x="48.26" y="34.29" rot="R180"/>
+<element name="R3" library="rcl" package="M1206" value="1uH" x="55.245" y="30.48" rot="R90"/>
 <element name="R4" library="rcl" package="M1206" value="150" x="55.245" y="25.4" rot="R90"/>
 <element name="R5" library="rcl" package="M1206" value="22" x="60.96" y="25.4" rot="R270"/>
-<element name="R6" library="rcl" package="M1206" value="1u" x="60.96" y="30.48" rot="R270"/>
+<element name="R6" library="rcl" package="M1206" value="1uH" x="60.96" y="30.48" rot="R270"/>
 <element name="U$1" library="minicircuits" package="DF782" value="PGA-103" x="56.515" y="38.735"/>
 <element name="X1" library="con-coax" package="J502-ND-142-0701-851/861" value="SMA" x="14.605" y="0" rot="R90">
@@
 <attribute name="MPN" value="142-0701-851" x="83.185" y="0" size="1.778" layer="27" rot="R90" display="off"/>
 </element>
-<element name="C15" library="rcl" package="C1206" value="1n" x="23.8125" y="26.3525" rot="R180"/>
-<element name="C16" library="rcl" package="C1206" value="1n" x="73.3425" y="26.035"/>
+<element name="C15" library="rcl" package="C1206" value="10n" x="23.8125" y="26.3525" rot="R180"/>
+<element name="C16" library="rcl" package="C1206" value="100n" x="73.3425" y="26.035"/>
 </elements>
 <signals>
