File: Relay Sequencer/Relay Sequencer.brd (EAGLE design)
At the start: 95.2 x 81.3 mm, 51 parts, among them IC1 MEGA16-A, IC2 ULN2003AD, IC3 7805DT, IC4 74HC244DW, K1 351, K2 351, K3 351, K4 351

Commit message: Reconfiguring Relays
Connections:
- removed net R2B: J4.2, K2.S1, K2.S2
- net +12V: now also K2.O1, K2.O2
- net GND: now also J4.2, K2.S1, K2.S2
Routing:
- net GND: track 374.2 -> 394.8 mm
- net R2B: track 14.3 -> 0.00 mm
- net +12V: track 371.6 -> 385.5 mm
- net N$12: track 6.35 -> 0.00 mm
- net N$11: track 5.72 -> 0.00 mm
Changed lines of the file:
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@@
 <rectangle x1="13.0175" y1="12.3825" x2="24.13" y2="21.9075" layer="30"/>
 <text x="38.4175" y="1.27" size="1.4224" layer="1" font="vector" ratio="16">SDL EME RELAY SEQUENCER - v1</text>
-<text x="53.0225" y="76.835" size="1.4224" layer="1" font="vector" ratio="16">RELAY</text>
+<text x="55.5625" y="78.74" size="1.4224" layer="1" font="vector" ratio="16">RELAY</text>
 <text x="64.77" y="76.835" size="1.4224" layer="1" font="vector" ratio="16">SEND</text>
 <text x="75.2475" y="76.835" size="1.4224" layer="1" font="vector" ratio="16">TX INH</text>
@@
 <wire x1="51.435" y1="57.785" x2="50.8" y2="57.15" width="1.016" layer="30"/>
 <wire x1="50.8" y1="57.15" x2="40.3225" y2="57.15" width="1.016" layer="30"/>
-<wire x1="53.6575" y1="73.66" x2="53.6575" y2="71.4375" width="1.016" layer="30"/>
-<wire x1="53.6575" y1="71.4375" x2="54.61" y2="70.485" width="1.016" layer="30"/>
+<wire x1="53.975" y1="73.3425" x2="53.975" y2="71.12" width="1.016" layer="30"/>
+<wire x1="53.975" y1="71.12" x2="54.61" y2="70.485" width="1.016" layer="30"/>
 <wire x1="54.61" y1="70.485" x2="54.61" y2="67.31" width="1.016" layer="30"/>
 <wire x1="54.61" y1="67.31" x2="62.23" y2="67.31" width="1.016" layer="30"/>
@@
 <wire x1="92.3925" y1="57.15" x2="82.55" y2="57.15" width="1.016" layer="30"/>
 <text x="41.275" y="76.835" size="1.4224" layer="1" font="vector" ratio="16">- +12V</text>
-<text x="48.5775" y="78.74" size="1.4224" layer="1" font="vector" ratio="16">LNA</text>
+<text x="42.8625" y="78.74" size="1.4224" layer="1" font="vector" ratio="16">LNA</text>
 <wire x1="48.26" y1="62.23" x2="24.765" y2="62.23" width="1.016" layer="30"/>
 <wire x1="24.765" y1="62.23" x2="23.495" y2="63.5" width="1.016" layer="30"/>
 <wire x1="42.545" y1="67.31" x2="37.1475" y2="67.31" width="1.016" layer="30"/>
+<wire x1="54.61" y1="62.23" x2="62.23" y2="62.23" width="1.016" layer="30"/>
+<text x="51.1175" y="78.74" size="1.4224" layer="1" font="vector" ratio="16">LNA</text>
+<text x="52.705" y="76.835" size="1.4224" layer="1" font="vector" ratio="16">- +12V</text>
 </plain>
 <attributes>
@@
 <wire x1="32.385" y1="68.58" x2="32.385" y2="73.5838" width="1.016" layer="16"/>
 <wire x1="32.385" y1="73.5838" x2="32.4612" y2="73.66" width="1.016" layer="16"/>
+<contactref element="J4" pad="2"/>
+<contactref element="K2" pad="S2"/>
+<contactref element="K2" pad="S1"/>
+<wire x1="62.23" y1="67.31" x2="54.61" y2="67.31" width="1.016" layer="16"/>
+<wire x1="54.61" y1="67.31" x2="54.61" y2="70.485" width="1.016" layer="16"/>
+<wire x1="54.61" y1="70.485" x2="53.975" y2="71.12" width="1.016" layer="16"/>
+<wire x1="53.975" y1="71.12" x2="53.975" y2="73.5838" width="1.016" layer="16"/>
+<wire x1="53.975" y1="73.5838" x2="53.8988" y2="73.66" width="1.016" layer="16"/>
+<wire x1="54.61" y1="67.31" x2="48.26" y2="67.31" width="1.016" layer="1"/>
 </signal>
 <signal name="N$1">
@@
 <wire x1="62.23" y1="52.07" x2="76.2" y2="52.07" width="1.016" layer="16"/>
 <wire x1="76.2" y1="52.07" x2="76.2" y2="49.53" width="1.016" layer="16"/>
+<contactref element="K2" pad="O1"/>
+<contactref element="K2" pad="O2"/>
+<wire x1="62.23" y1="62.23" x2="54.61" y2="62.23" width="1.016" layer="16"/>
+<wire x1="54.61" y1="62.23" x2="48.26" y2="62.23" width="1.016" layer="1"/>
 </signal>
 <signal name="EVENT_1">
@@
 <wire x1="57.785" y1="71.12" x2="57.785" y2="73.5838" width="1.016" layer="16"/>
 <wire x1="57.785" y1="73.5838" x2="57.8612" y2="73.66" width="1.016" layer="16"/>
-</signal>
-<signal name="R2B">
-<contactref element="K2" pad="S1"/>
-<contactref element="K2" pad="S2"/>
-<contactref element="J4" pad="2"/>
-<wire x1="54.61" y1="67.31" x2="62.23" y2="67.31" width="1.016" layer="16"/>
-<wire x1="53.8988" y1="73.66" x2="53.8988" y2="71.1962" width="1.016" layer="16"/>
-<wire x1="53.8988" y1="71.1962" x2="54.61" y2="70.485" width="1.016" layer="16"/>
-<wire x1="54.61" y1="70.485" x2="54.61" y2="67.31" width="1.016" layer="16"/>
 </signal>
 <signal name="R3A">
@@
 <wire x1="86.995" y1="34.29" x2="83.7692" y2="34.29" width="0.6096" layer="1"/>
 </signal>
-<signal name="N$11">
-<wire x1="53.34" y1="79.375" x2="58.42" y2="79.375" width="0.4064" layer="1"/>
-<wire x1="58.42" y1="79.375" x2="58.42" y2="78.74" width="0.4064" layer="1"/>
-</signal>
-<signal name="N$12">
-<wire x1="47.625" y1="79.375" x2="41.91" y2="79.375" width="0.4064" layer="1"/>
-<wire x1="41.91" y1="79.375" x2="41.91" y2="78.74" width="0.4064" layer="1"/>
-</signal>
 </signals>

Commit message: Revalue the components
Parts:
- C1, C5: value (none) -> 22p
- C10, C13, C14, C15, C6: value (none) -> 100n
- C11: value (none) -> 1u
- C12, C3, C4, C7, C8, C9: value (none) -> 10n
- C2: value (none) -> 1n
- R1: value (none) -> 10k
- R2, R3, R4, R5, R6, R7: value (none) -> 560
Changed lines of the file:
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@@
 </autorouter>
 <elements>
-<element name="C1" library="rcl" package="C1206" value="" x="56.515" y="9.525" rot="R270"/>
-<element name="C12" library="rcl" package="E5-13" value="" x="22.86" y="27.94" rot="R90"/>
-<element name="C13" library="rcl" package="C1206" value="" x="6.35" y="19.685" rot="R180"/>
-<element name="C14" library="rcl" package="C1206" value="" x="6.35" y="14.605" rot="R180"/>
-<element name="C2" library="rcl" package="C1206" value="" x="65.405" y="34.29" rot="R90"/>
-<element name="C3" library="rcl" package="C1206" value="" x="76.835" y="24.765"/>
-<element name="C5" library="rcl" package="C1206" value="" x="70.485" y="9.525" rot="R270"/>
-<element name="C6" library="rcl" package="C1206" value="" x="46.355" y="22.86" rot="R180"/>
-<element name="C8" library="rcl" package="C1206" value="" x="46.355" y="12.065" rot="R180"/>
-<element name="C9" library="rcl" package="C1206" value="" x="9.525" y="51.435" rot="R180"/>
-<element name="C10" library="rcl" package="C1206" value="" x="13.335" y="31.115" rot="R180"/>
-<element name="C11" library="rcl" package="E5-8,5" value="" x="6.35" y="27.94" rot="R90"/>
+<element name="C1" library="rcl" package="C1206" value="22p" x="56.515" y="9.525" rot="R270"/>
+<element name="C12" library="rcl" package="E5-13" value="10n" x="22.86" y="27.94" rot="R90"/>
+<element name="C13" library="rcl" package="C1206" value="100n" x="6.35" y="19.685" rot="R180"/>
+<element name="C14" library="rcl" package="C1206" value="100n" x="6.35" y="14.605" rot="R180"/>
+<element name="C2" library="rcl" package="C1206" value="1n" x="65.405" y="34.29" rot="R90"/>
+<element name="C3" library="rcl" package="C1206" value="10n" x="76.835" y="24.765"/>
+<element name="C5" library="rcl" package="C1206" value="22p" x="70.485" y="9.525" rot="R270"/>
+<element name="C6" library="rcl" package="C1206" value="100n" x="46.355" y="22.86" rot="R180"/>
+<element name="C8" library="rcl" package="C1206" value="10n" x="46.355" y="12.065" rot="R180"/>
+<element name="C9" library="rcl" package="C1206" value="10n" x="9.525" y="51.435" rot="R180"/>
+<element name="C10" library="rcl" package="C1206" value="100n" x="13.335" y="31.115" rot="R180"/>
+<element name="C11" library="rcl" package="E5-8,5" value="1u" x="6.35" y="27.94" rot="R90"/>
 <element name="D1" library="diode" package="DO35-10" value="1N400x" x="28.575" y="42.545" rot="R270"/>
 <element name="D2" library="diode" package="DO35-10" value="1N400x" x="23.495" y="68.58" rot="R90"/>
@@
 <attribute name="OC_NEWARK" value="unknown" x="63.5" y="9.525" size="1.778" layer="27" display="off"/>
 </element>
-<element name="R1" library="rcl" package="M1206" value="" x="46.355" y="15.24" rot="R180"/>
-<element name="R2" library="rcl" package="M1206" value="" x="46.355" y="39.37"/>
-<element name="R3" library="rcl" package="M1206" value="" x="46.355" y="34.925"/>
-<element name="R4" library="rcl" package="M1206" value="" x="46.355" y="30.48"/>
-<element name="R5" library="rcl" package="M1206" value="" x="46.355" y="26.035"/>
-<element name="R6" library="rcl" package="M1206" value="" x="46.355" y="19.685"/>
-<element name="R7" library="rcl" package="M1206" value="" x="11.1125" y="10.16" rot="R90"/>
+<element name="R1" library="rcl" package="M1206" value="10k" x="46.355" y="15.24" rot="R180"/>
+<element name="R2" library="rcl" package="M1206" value="560" x="46.355" y="39.37"/>
+<element name="R3" library="rcl" package="M1206" value="560" x="46.355" y="34.925"/>
+<element name="R4" library="rcl" package="M1206" value="560" x="46.355" y="30.48"/>
+<element name="R5" library="rcl" package="M1206" value="560" x="46.355" y="26.035"/>
+<element name="R6" library="rcl" package="M1206" value="560" x="46.355" y="19.685"/>
+<element name="R7" library="rcl" package="M1206" value="560" x="11.1125" y="10.16" rot="R90"/>
 <element name="J2" library="con-amp" package="1X2MTA" value="" x="16.51" y="73.66"/>
-<element name="C4" library="rcl" package="C1206" value="" x="29.845" y="51.435"/>
-<element name="C7" library="rcl" package="C1206" value="" x="76.835" y="20.955"/>
+<element name="C4" library="rcl" package="C1206" value="10n" x="29.845" y="51.435"/>
+<element name="C7" library="rcl" package="C1206" value="10n" x="76.835" y="20.955"/>
 <element name="IC4" library="74xx-eu" package="SO20W" value="74HC244DW" x="78.74" y="38.735" rot="R270"/>
-<element name="C15" library="rcl" package="C1206" value="" x="82.2325" y="46.6725" rot="R180"/>
+<element name="C15" library="rcl" package="C1206" value="100n" x="82.2325" y="46.6725" rot="R180"/>
 </elements>
 <signals>
