File: Test Arduino Shield/Test Arduino Shield.brd (EAGLE design)
At the start: 68.6 x 53.3 mm, 15 parts, among them M1 ARDUINO_R3_ICSP

Commit message: Adding Dorji Lib
Parts:
- added U$2: (no value), dorji:DRA818A
Changed lines of the file:
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@@
 <?xml version="1.0" encoding="utf-8"?>
 <!DOCTYPE eagle SYSTEM "eagle.dtd">
-<eagle version="7.2.0">
+<eagle version="7.7.0">
 <drawing>
 <settings>
@@
 <setting verticaltext="up"/>
 </settings>
-<grid distance="0.01" unitdist="inch" unit="inch" style="lines" multiple="1" display="no" altdistance="0.025" altunitdist="inch" altunit="inch"/>
+<grid distance="0.01" unitdist="inch" unit="mm" style="dots" multiple="1" display="yes" altdistance="0.025" altunitdist="inch" altunit="inch"/>
 <layers>
 <layer number="1" name="Top" color="4" fill="1" visible="yes" active="yes"/>
@@
 <hole x="66.5581" y="35.5143" drill="2.2"/>
 <text x="2.794" y="7.366" size="1.27" layer="21" font="vector" ratio="12">Reset</text>
+<dimension x1="41.656" y1="50.8" x2="45.72" y2="50.8" x3="43.688" y3="53.848" textsize="1.778" layer="16"/>
+<dimension x1="63.5" y1="50.8" x2="63.5" y2="2.54" x3="72.898" y3="26.67" textsize="1.778" layer="16"/>
+<dimension x1="45.72" y1="2.54" x2="50.8" y2="2.54" x3="48.26" y3="-3.048" textsize="1.778" layer="16"/>
 </plain>
 <attributes>
@@
 <element name="U$1" library="adafruit" package="1X10-BIG" value="PINHD-1X10" x="30.226" y="46.99"/>
 <element name="U$36" library="microbuilder" package="ADAFRUIT_9MM" value="" x="10.668" y="42.672" rot="MR270"/>
+<element name="U$2" library="dorji" package="DRA818A" value="" x="-18.034" y="30.48" rot="R180"/>
 </elements>
 <signals>
@@
 <contactref element="M1" pad="GND@1"/>
 <contactref element="M1" pad="GND@2"/>
-<contactref element="M1" pad="GND@3"/>
-<contactref element="M1" pad="GND@1"/>
 <contactref element="M1" pad="GND"/>
 <contactref element="JP1" pad="2"/>
