File: Test Arduino Shield/Test Arduino Shield.sch (EAGLE design)
At the start: 14 parts, among them M1 ARDUINO_R3_ICSP

Commit message: Adding Dorji Lib
Parts:
- added U$2: (no value), dorji:DRA818A
Changed lines of the file:
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@@
 <?xml version="1.0" encoding="utf-8"?>
 <!DOCTYPE eagle SYSTEM "eagle.dtd">
-<eagle version="7.2.0">
+<eagle version="7.7.0">
 <drawing>
 <settings>
@@
 <part name="JP1" library="carduino" deviceset="PINHD-1X8" device="BIG"/>
 <part name="U$1" library="adafruit" deviceset="PINHD-1X10" device=""/>
+<part name="U$2" library="dorji" deviceset="DRA818A" device=""/>
 </parts>
 <sheets>
@@
 <instance part="JP1" gate="G$1" x="66.04" y="20.32" rot="R270"/>
 <instance part="U$1" gate="G$1" x="53.34" y="104.14" rot="R90"/>
+<instance part="U$2" gate="G$1" x="-38.1" y="76.2"/>
 </instances>
 <busses>
